Commit message: adding Docker environment

File: motion_policy_configs/ur3e/ur3e_gripper.urdf (robot description, URDF)
Before this commit: robot ur3e, 15 links, 14 joints
Links:
- link single_base: geometry collision mesh filename=zimmer_gripper/zimmer_description/meshes/collision/zimmer_b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 scale=0.001 0.001 0.001; visual mesh filename=zimmer_gripper/zimmer_description/meshes/visual/gripper_bod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
- link single_finger_left: geometry collision mesh filename=zimmer_gripper/zimmer_description/meshes/collision/Left_Fin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 scale=0.001 0.001 0.001; visual mesh filename=zimmer_gripper/zimmer_description/meshes/visual/left_finger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
- link single_finger_right: geometry collision mesh filename=zimmer_gripper/zimmer_description/meshes/collision/Right_Fi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 scale=0.001 0.001 0.001; visual mesh filename=zimmer_gripper/zimmer_description/meshes/visual/right_finge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
Joints:
- joint gripper_center_joint: origin xyz=0.0 0.0 0.1 rpy=0 0 0 -> xyz=0.0 0.0 0.1 rpy=0 0 0.401426
- joint single_to_base: origin xyz=0 0.0 0.0 rpy=0 0 0.23 -> xyz=0 0.0 0.0 rpy=0 0 0.401426
